File: KiCAD/@home/@home.kicad_sch (KiCad schematic)
At the start: 4 parts, among them J1 Raspberry_Pi_2_3, J2 Conn_01x04_Socket

Commit message: Android app developing and a tutorial for when i connect the rpi to the app
Parts:
- J1: value Raspberry_Pi_2_3 -> Raspberry_Pi4
Changed lines of the file:
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@@
 			)
 		)
-		(property "Value" "Raspberry_Pi_2_3"
+		(property "Value" "Raspberry_Pi4"
 			(at 59.2933 95.25 0)
 			(effects
