File: KiCAD/weather station/weather station.kicad_pcb (KiCad board)
At the start: 4 copper layers, 55 x 55.5 mm, 14 parts, among them J2 RS485 ANEMOMETER, J4 RS485 WIND DIRECTION, U1 PTN78000H_EUS-5, U2 MAX485E, U3 DHT22

Commit message: PCB update and firmware update
Parts:
- added J6: FS100A, Connector_PinHeader_2.54mm:PinHeader_1x03_P2.54mm_Vertical, F.Cu at (79.0, 87.5)
- added R4: 2K2, Resistor_THT:R_Axial_DIN0204_L3.6mm_D1.6mm_P5.08mm_Horizontal, F.Cu at (71.0, 89.0)
- added U4: DS18B20-, Connector_PinHeader_2.54mm:PinHeader_1x03_P2.54mm_Vertical, F.Cu at (85.5, 87.4)
- added U5: DS18B20, Connector_PinHeader_2.54mm:PinHeader_1x03_P2.54mm_Vertical, F.Cu at (87.0, 75.0)
Connections:
- A1 pad 11: Net-(A1-D8) -> RO
- A1 pad 12: Net-(A1-D9) -> DI
- A1 pad 5: unconnected-(A1-D2-Pad5) -> Net-(A1-D2)
- A1 pad 6: unconnected-(A1-D3-Pad6) -> Net-(A1-D3)
- U2 pad 1: Net-(A1-D8) -> D8
- U2 pad 4: Net-(A1-D9) -> D9
Routing:
- net Net-(A1-D2): track 0.00 -> 76.7 mm
- net (no net): track 0.00 -> 72.7 mm
- net Net-(A1-D3): track 0.00 -> 57.4 mm
- net Net-(A1-+5V): track 78.2 -> 122.0 mm
- net Net-(A1-D8): track 36.6 -> 0.00 mm
- net Net-(A1-D9): track 36.1 -> 0.00 mm
- net GND: track 144.9 -> 163.0 mm
- net +12V: track 86.0 -> 95.0 mm

Commit message: Android app developing and a tutorial for when i connect the rpi to the app
Parts:
- U4: value DS18B20- -> DS18B20
Connections:
- A1 pad 11: RO -> D8
- A1 pad 12: DI -> D9
Routing:
- net (no net): track 72.7 -> 0.00 mm
- net D8: track 0.00 -> 36.4 mm
- net D9: track 0.00 -> 34.1 mm
