File: KiCAD/weather station/weather station.kicad_sch (KiCad schematic)
At the start: 18 parts, among them J1 RS485 ANEMOMETER, J2 RS485 ANEMOMETER, J3 RS485 WIND DIRECTION, J4 RS485 WIND DIRECTION, J5 SDLA12TA, U1 PTN78000H_EUS-5, U2 MAX485E, U3 DHT22

Commit message: PCB update and firmware update
Parts:
- added J6: FS100A, Connector_PinHeader_2.54mm:PinHeader_1x03_P2.54mm_Vertical, symbol Connector:Conn_01x03_Pin
- added R4: 2K2, Resistor_THT:R_Axial_DIN0204_L3.6mm_D1.6mm_P5.08mm_Horizontal, symbol Device:R
- added U4, U5: DS18B20, Connector_PinHeader_2.54mm:PinHeader_1x03_P2.54mm_Vertical, symbol Sensor_Temperature:DS18B20
Connections:
- net +12V: now also J6.1 (Pin_1)
- net GND: now also U4.1 (GND), U5.1 (GND)
- net at A1.27 (+5V), C2.1, R3.2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: now also R4.1, U4.3 (V_{DD}), U5.3 (V_{DD})
- net at A1.5 (D2): now also R4.2, U4.2 (DQ), U5.2 (DQ)
- net at A1.6 (D3): now also J6.2 (Pin_2)
- no-connect marks 23 -> 22

Commit message: Android app developing and a tutorial for when i connect the rpi to the app
Connections:
- net DI is gone; now on net D9: A1.12 (D9)
- net RO is gone; now on net D8: A1.11 (D8)
Changed lines of the file:
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@@
+	)
+	(junction
+		(at 17.78 67.31)
+		(diameter 0)
+		(color 0 0 0 0)
 	)
 	(junction
@@
 	(wire
 		(pts
+			(xy 13.97 96.52) (xy 43.18 96.52)
+		)
+		(stroke
+			(width 0)
+			(type default)
+		)
+	)
+	(wire
+		(pts
 			(xy 125.73 25.4) (xy 125.73 20.32)
 		)
@@
 	(wire
 		(pts
-			(xy 41.91 99.06) (xy 43.18 99.06)
-		)
-		(stroke
-			(width 0)
-			(type default)
-		)
-	)
-	(wire
-		(pts
 			(xy 102.87 85.09) (xy 85.09 85.09)
 		)
@@
 	(wire
 		(pts
+			(xy 17.78 99.06) (xy 17.78 67.31)
+		)
+		(stroke
+			(width 0)
+			(type default)
+		)
+	)
+	(wire
+		(pts
 			(xy 55.88 57.15) (xy 46.99 57.15)
 		)
@@
 	(wire
 		(pts
+			(xy 13.97 96.52) (xy 13.97 57.15)
+		)
+		(stroke
+			(width 0)
+			(type default)
+		)
+	)
+	(wire
+		(pts
 			(xy 46.99 57.15) (xy 46.99 49.53)
 		)
@@
 	(wire
 		(pts
+			(xy 17.78 99.06) (xy 43.18 99.06)
+		)
+		(stroke
+			(width 0)
+			(type default)
+		)
+	)
+	(wire
+		(pts
 			(xy 48.26 20.32) (xy 49.53 20.32)
 		)
@@
 	(wire
 		(pts
-			(xy 16.51 57.15) (xy 17.78 57.15)
-		)
-		(stroke
-			(width 0)
-			(type default)
-		)
-	)
-	(wire
-		(pts
 			(xy 38.1 53.34) (xy 41.91 53.34)
 		)
@@
 	(wire
 		(pts
+			(xy 13.97 57.15) (xy 17.78 57.15)
+		)
+		(stroke
+			(width 0)
+			(type default)
+		)
+	)
+	(wire
+		(pts
 			(xy 54.61 55.88) (xy 55.88 55.88)
 		)
@@
 		)
 		(stroke
-			(width 0)
-			(type default)
-		)
-	)
-	(wire
-		(pts
-			(xy 41.91 96.52) (xy 43.18 96.52)
-		)
-		(stroke
